Commit message: Implemented full simulation with gazebo_control, errors were found with ros2_control, related robably with the URDF structure, further inspection necessary, consider fork.

File: src/f112th_sim_2501_camel/description/properties.xacro (robot description, xacro)
@@ -14,4 +14,5 @@
         <color rgba= "0 0 0 1"/>
     </material>
+    <!-- Color Definitions -->
     <gazebo reference="chassis">
         <material>Gazebo/White</material>
@@ -26,3 +27,8 @@
         <material>Gazebo/Blue</material>
     </gazebo>
+    <gazebo reference="caster_wheel">
+        <material>Gazebo/Black</material>
+        <mu1 value="0.001"/>
+        <mu2 value="0.001"/>
+    </gazebo>
 </robot>

File: src/f112th_sim_2501_camel/description/robot.urdf.xacro (robot description, xacro)
@@ -1,8 +1,9 @@
 <?xml version="1.0"?>
-<robot xmlns:xacro="http://www.ros.org/wiki/xacro" name="Diffdrive">
+<robot xmlns:xacro="http://www.ros.org/wiki/xacro" name = "rodolfo">
     <!-- Example link -->
     <xacro:include filename="properties.xacro"/>
     <xacro:include filename="robot_core.xacro"/>
-    <xacro:include filename="inertial_macros.xacro"/>
+    <xacro:include filename="lidar.xacro"/>
+    <!-- <xacro:include filename="ros2_control.xacro"/> -->
     <xacro:include filename="gazebo_control.xacro"/>
 </robot>

File: src/f112th_sim_2501_camel/description/robot_core.xacro (robot description, xacro)
@@ -17,5 +17,4 @@
                 <box size="0.3 0.3 0.15"/>
             </geometry>
-            <material name="white"/>
         </visual>
         <collision>
@@ -25,5 +24,5 @@
             </geometry>
         </collision>
-        <xacro:inertial_box mass="0.5" x="0.3" y="0.3" z="0.15">
+        <xacro:inertial_box mass="0.8" x="0.3" y="0.3" z="0.15">
             <origin xyz="0.15 0 0.075" rpy="0 0 0"/>
         </xacro:inertial_box>
@@ -42,11 +41,10 @@
                 <cylinder radius="0.05" length="0.04"/>
             </geometry>
-            <material name="blue"/>
         </visual>
-        <collision>
-            <geometry>
-                <cylinder radius="0.05" length="0.04"/>
-            </geometry>
-        </collision>
+	      <collision>
+	          <geometry>
+	              <sphere radius="0.05"/>
+	          </geometry>
+	      </collision>
         <xacro:inertial_cylinder mass="0.1" length="0.04" radius="0.05">
             <origin xyz="0 0 0" rpy="0 0 0"/>
@@ -66,11 +64,10 @@
                 <cylinder radius="0.05" length="0.04"/>
             </geometry>
-            <material name="blue"/>
         </visual>
-        <collision>
-            <geometry>
-                <cylinder radius="0.05" length="0.04"/>
-            </geometry>
-        </collision>
+	      <collision>
+	          <geometry>
+	              <sphere radius="0.05"/>
+	          </geometry>
+	      </collision>
         <xacro:inertial_cylinder mass="0.1" length="0.04" radius="0.05">
             <origin xyz="0 0 0" rpy="0 0 0"/>
@@ -85,10 +82,4 @@
     <!-- caster wheel link -->
     <link name="caster_wheel">
-        <visual>
-            <geometry>
-                <sphere radius="0.05"/>
-            </geometry>
-            <material name="black"/>
-        </visual>
         <collision>
             <geometry>
@@ -96,4 +87,9 @@
             </geometry>
         </collision>
+        <visual>
+            <geometry>
+                <sphere radius="0.05"/>
+            </geometry>
+        </visual>
         <xacro:inertial_sphere mass="0.1" radius="0.05">
             <origin xyz="0 0 0" rpy="0 0 0"/>
