Commit message: Entrega realizada

File: src/f112th_sim_2501_camel/description/ack_drive/bot_base.xacro (robot description, xacro)
@@ -1,11 +1,11 @@
 <?xml version="1.0"?>
 <robot xmlns:xacro="http://www.ros.org/wiki/xacro">
-    <xacro:property name="body_mass" value="0.7" />
+    <xacro:property name="body_mass" value="0.3" />
     <xacro:property name="body_width" value="0.3" />
     <xacro:property name="body_length" value="0.10" />
     <xacro:property name="body_depth" value="0.75" />
     <xacro:property name="wheel_radius" value="0.1" />
-    <xacro:property name="wheel_thickness" value="0.1" />
-    <xacro:property name="wheel_mass" value="0.3" />
+    <xacro:property name="wheel_thickness" value="0.05  " />
+    <xacro:property name="wheel_mass" value="0.8" />
     <xacro:property name="steering_mass" value="0.01" />
     <!-- BASE -->

File: src/f112th_sim_2501_camel/description/ack_drive/bot_base_mine.xacro (robot description, xacro)
@@ -1,12 +1,12 @@
 <?xml version="1.0"?>
 <robot xmlns:xacro="http://www.ros.org/wiki/xacro">
-    <xacro:property name="body_mass" value="25.0" />
+    <xacro:property name="body_mass" value="0.5" />
     <xacro:property name="body_width" value="0.3" />
     <xacro:property name="body_length" value="0.10" />
     <xacro:property name="body_depth" value="0.5" />
     <xacro:property name="wheel_radius" value="0.06" />
-    <xacro:property name="wheel_thickness" value="0.06" />
-    <xacro:property name="wheel_mass" value="0.01" />
-    <xacro:property name="steering_mass" value="0.01" />
+    <xacro:property name="wheel_thickness" value="0.01" />
+    <xacro:property name="wheel_mass" value="5.0" />
+    <xacro:property name="steering_mass" value="5.00" />
     <!-- BASE -->
     <link name="base_footprint">
